File: pcb/eink_digit_clk.kicad_pcb (KiCad board)
At the start: 2 copper layers, 53 x 93 mm, 56 parts, among them J1 24-pin-epd-fpc, J2 USB_C_Receptacle_USB2.0_16P, J3 Conn_01x02, Q1 AO3400, Q2 AO3401, SW1 Boot, SW2 Reset, U1 ESP32-C6-WROOM-1, U2 TP4057, U3 HT7833_SOT89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

Commit message: Fix issues in schematic/pcb
Parts:
- added C21: 10u, Capacitor_SMD:C_0805_2012Metric, F.Cu at (131.0, 104.7)
- added U4: HT7833_SOT89, Package_TO_SOT_SMD:SOT-89-3, F.Cu at (90.3, 133.2)
Connections:
- U1 pad 10: unconnected-(U1-GPIO8-Pad10) -> +3V3
Routing:
- net +3V3: track 125.2 -> 138.7 mm, vias 6 -> 8
- net Net-(D4-K): track 14.8 -> 19.9 mm
- net GND: track 86.2 -> 91.1 mm
Other:
- board text added: "EINK CLOCK DIGIT V1.1 (C) SPRITESMODS 2024"
- board text removed: "EINK CLOCK DIGIT V1.0 (C) SPRITESMODS 2024"
