File: pcb/eink_digit_clk.kicad_sch (KiCad schematic)
At the start: 56 parts, among them J1 24-pin-epd-fpc, J2 USB_C_Receptacle_USB2.0_16P, J3 Conn_01x02, Q1 AO3400, Q2 AO3401, SW1 Boot, SW2 Reset, U1 ESP32-C6-WROOM-1, U2 TP4057, U3 HT7833_SOT89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

Commit message: It works, but with ntp sync, so the digits will drift apart
Other:
- note added: "Issue: GPIO8 should be high for download mode"
Changed lines of the file:
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@@
+    (effects (font (size 1.27 1.27)) (justify left bottom))
+  )
+  (text "Issue: GPIO8\nshould be high\nfor download mode" (at 176.53 114.3 0)
     (effects (font (size 1.27 1.27)) (justify left bottom))
   )

Commit message: Fix issues in schematic/pcb
Parts:
- added C21: 10u, Capacitor_SMD:C_0805_2012Metric, symbol Device:C_Small
- added U4: HT7833_SOT89, Package_TO_SOT_SMD:SOT-89-3, symbol Jeroens lib:HT7833_SOT89
- C17, C18: value 5p -> 15p
Connections:
- net +3V3: now also U1.10 (GPIO8), C21.1, U4.3 (VOUT)
- net GND: now also C21.2, U4.1 (GND)
- net at C1.1, D4.1 (K), Q2.2 (S)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: now also U4.2 (VIN)
- no-connect marks 15 -> 14
Other:
- note added: "Note: add U4 in case of brownout issues"
- note added: "may need to tweak R9, C18, C17 if RTC doesn't start"
- note removed: "Issue: GPIO8 should be high for download mode"
- note removed: "Use LP GPIO 2-7, reserve 5 if needed (LPTxD)"
- moved on the sheet: C1, C10, C11, C12, C13, C14, C15, C16, C17, C18, C19, C2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
